Commit message: Updated feetech ros2 driver.

File: so101_description/urdf/ros2_control/so101_ros2_control.xacro (robot description, xacro)
@@ -1,6 +1,7 @@
 <?xml version="1.0"?>
 <robot xmlns:xacro="http://www.ros.org/wiki/xacro">
-    <xacro:macro name="so101_control_joint" params="variant joint">
+    <xacro:macro name="so101_control_joint" params="variant joint id">
         <joint name="${joint}">
+            <param name="id">${id}</param>
             <!-- follower can be commanded; leader is state-only -->
             <xacro:if value="${variant == 'follower'}">
@@ -33,10 +34,10 @@
             </hardware>
             <!-- arm joints -->
-            <xacro:so101_control_joint  variant="${variant}" joint="shoulder_pan"/>
-            <xacro:so101_control_joint  variant="${variant}" joint="shoulder_lift"/>
-            <xacro:so101_control_joint  variant="${variant}" joint="elbow_flex"/>
-            <xacro:so101_control_joint  variant="${variant}" joint="wrist_flex"/>
-            <xacro:so101_control_joint  variant="${variant}" joint="wrist_roll"/>
-            <xacro:so101_control_joint  variant="${variant}" joint="gripper"/>
+            <xacro:so101_control_joint variant="${variant}" joint="shoulder_pan"  id="1"/>
+            <xacro:so101_control_joint variant="${variant}" joint="shoulder_lift" id="2"/>
+            <xacro:so101_control_joint variant="${variant}" joint="elbow_flex"   id="3"/>
+            <xacro:so101_control_joint variant="${variant}" joint="wrist_flex"   id="4"/>
+            <xacro:so101_control_joint variant="${variant}" joint="wrist_roll"   id="5"/>
+            <xacro:so101_control_joint variant="${variant}" joint="gripper"      id="6"/>
         </ros2_control>
     </xacro:macro>
