Commit message: add simulated arms bringup, add teleop with keyboard sim

File: so101_description/urdf/end_effectors/so101_ee_common.xacro (robot description, xacro)
@@ -25,4 +25,5 @@
       <axis xyz="0 0 1"/>
       <limit effort="10" velocity="10" lower="-2.74385" upper="2.84121"/>
+      <dynamics damping="0.12" friction="0.02"/>
     </joint>
     <xacro:if value="${add_transmission}">

File: so101_description/urdf/end_effectors/so101_ee_follower.xacro (robot description, xacro)
@@ -30,4 +30,5 @@
       <axis xyz="0 0 1"/>
       <limit effort="10" velocity="10" lower="-0.174533" upper="1.74533"/>
+      <dynamics damping="0.08" friction="0.01"/>
     </joint>
     <!-- follower-only motor6 transmission (optional) -->

File: so101_description/urdf/end_effectors/so101_ee_leader.xacro (robot description, xacro)
@@ -32,4 +32,5 @@
       <axis xyz="0 0 1"/>
       <limit effort="10" velocity="10" lower="-0.174533" upper="1.74533"/>
+      <dynamics damping="0.08" friction="0.01"/>
     </joint>
     <xacro:so101_wrist_roll_joint

File: so101_description/urdf/ros2_control/so101_ros2_control.xacro (robot description, xacro)
@@ -1,9 +1,9 @@
 <?xml version="1.0"?>
 <robot xmlns:xacro="http://www.ros.org/wiki/xacro">
-    <xacro:macro name="so101_control_joint" params="variant joint id">
+    <xacro:macro name="so101_control_joint" params="variant hardware_type joint id">
         <joint name="${joint}">
             <param name="id">${id}</param>
             <!-- follower can be commanded; leader is state-only -->
-            <xacro:if value="${variant == 'follower'}">
+            <xacro:if value="${variant == 'follower' or hardware_type == 'gazebo'}">
                 <command_interface name="position"/>
                 <param name="p_coefficient">16</param>
@@ -39,12 +39,15 @@
                     <param name="joint_config_file">${joint_config_file}</param>
                 </xacro:if>
+                    <xacro:if value="${hardware_type == 'gazebo'}">
+                        <plugin>gz_ros2_control/GazeboSimSystem</plugin>
+                    </xacro:if>
             </hardware>
             <!-- arm joints -->
-            <xacro:so101_control_joint variant="${variant}" joint="shoulder_pan"  id="1"/>
-            <xacro:so101_control_joint variant="${variant}" joint="shoulder_lift" id="2"/>
-            <xacro:so101_control_joint variant="${variant}" joint="elbow_flex"   id="3"/>
-            <xacro:so101_control_joint variant="${variant}" joint="wrist_flex"   id="4"/>
-            <xacro:so101_control_joint variant="${variant}" joint="wrist_roll"   id="5"/>
-            <xacro:so101_control_joint variant="${variant}" joint="gripper"      id="6"/>
+                <xacro:so101_control_joint variant="${variant}" hardware_type="${hardware_type}" joint="shoulder_pan"  id="1"/>
+                <xacro:so101_control_joint variant="${variant}" hardware_type="${hardware_type}" joint="shoulder_lift" id="2"/>
+                <xacro:so101_control_joint variant="${variant}" hardware_type="${hardware_type}" joint="elbow_flex"   id="3"/>
+                <xacro:so101_control_joint variant="${variant}" hardware_type="${hardware_type}" joint="wrist_flex"   id="4"/>
+                <xacro:so101_control_joint variant="${variant}" hardware_type="${hardware_type}" joint="wrist_roll"   id="5"/>
+                <xacro:so101_control_joint variant="${variant}" hardware_type="${hardware_type}" joint="gripper"      id="6"/>
         </ros2_control>
     </xacro:macro>

File: so101_description/urdf/so101_arm.urdf.xacro (robot description, xacro)
@@ -8,4 +8,9 @@
   <xacro:arg name="usb_port" default="/dev/ttyUSB0"/>
   <xacro:arg name="joint_config_file" default=""/>
+  <xacro:arg name="controller_config_file" default=""/>
+  <xacro:arg name="ros_namespace" default=""/>
+  <xacro:arg name="controller_manager_name" default="controller_manager"/>
+  <xacro:arg name="sim_hold_joints" default="true"/>
+  <xacro:arg name="sim_position_proportional_gain" default="0.35"/>
   <!-- Camera args -->
   <xacro:arg name="enable_static_cam" default="false"/>
@@ -18,4 +23,5 @@
   <xacro:property name="use_ros2_control" value="$(arg use_ros2_control)"/>
   <xacro:property name="variant" value="$(arg variant)"/>
+  <xacro:property name="hardware_type" value="$(arg hardware_type)"/>
   <xacro:property name="enable_static_cam" value="$(arg enable_static_cam)"/>
   <xacro:property name="enable_wrist_cam" value="$(arg enable_wrist_cam)"/>
@@ -28,4 +34,5 @@
   <xacro:include filename="$(find so101_description)/urdf/ros2_control/so101_ros2_control.xacro"/>
   <xacro:include filename="$(find so101_description)/urdf/so101_cameras.xacro"/>
+  <xacro:include filename="$(find so101_description)/urdf/so101_gazebo.xacro"/>
   <xacro:so101_materials/>
   <xacro:so101_arm_common
@@ -49,4 +56,13 @@
       joint_config_file="$(arg joint_config_file)"
       system_name="SO101_${variant}_SYSTEM"/>
+    <xacro:if value="${hardware_type == 'gazebo'}">
+      <xacro:so101_gazebo_world_fixed_joint/>
+      <xacro:so101_gazebo_control_plugin
+        namespace="$(arg ros_namespace)"
+        controller_config_file="$(arg controller_config_file)"
+        controller_manager_name="$(arg controller_manager_name)"
+        hold_joints="$(arg sim_hold_joints)"
+        position_proportional_gain="$(arg sim_position_proportional_gain)"/>
+    </xacro:if>
   </xacro:if>
   <!-- Cameras (opt-in via enable_static_cam / enable_wrist_cam) -->

File: so101_description/urdf/so101_arm_common.xacro (robot description, xacro)
@@ -78,4 +78,5 @@
       <axis xyz="0 0 1"/>
       <limit effort="10" velocity="10" lower="-1.91986" upper="1.91986"/>
+      <dynamics damping="0.25" friction="0.05"/>
     </joint>
     <joint name="shoulder_lift" type="revolute">
@@ -85,4 +86,5 @@
       <axis xyz="0 0 1"/>
       <limit effort="10" velocity="10" lower="-1.74533" upper="1.74533"/>
+      <dynamics damping="0.25" friction="0.05"/>
     </joint>
     <joint name="elbow_flex" type="revolute">
@@ -92,4 +94,5 @@
       <axis xyz="0 0 1"/>
       <limit effort="10" velocity="10" lower="-1.69" upper="1.69"/>
+      <dynamics damping="0.2" friction="0.04"/>
     </joint>
     <joint name="wrist_flex" type="revolute">
@@ -99,4 +102,5 @@
       <axis xyz="0 0 1"/>
       <limit effort="10" velocity="10" lower="-1.65806" upper="1.65806"/>
+      <dynamics damping="0.15" friction="0.03"/>
     </joint>
     <!-- OPTIONAL transmissions motor1..motor4 -->
